File: Hardware/Hardware.kicad_sch (KiCad schematic)
At the start: 38 parts, among them J1 Conn_01x04, J4 Conn_01x04, Q1 MMBT2222A, SW1 SW_Push, U1 STM32WB55RGVx, U4 BME280, Y1 32kHz768, Y2 32MHz

Commit message: [FOOTPRINT ASSIGNMENT] : Ajout des footprints à chaque élément
Parts:
- BZ1: footprint (none) -> Buzzer_Beeper:Buzzer_12x9.5RM7.6
- C1, C10, C12, C15, C16, C21, C3, C4, C5, C6, C7, C8, C9: footprint (none) -> Capacitor_SMD:C_0402_1005Metric
- C11, C13, C14, C2: footprint (none) -> Capacitor_SMD:C_0603_1608Metric
- D2, D3, D4: footprint (none) -> LED_THT:LED_D3.0mm
- J1, J4: footprint (none) -> Connector_PinHeader_1.00mm:PinHeader_1x04_P1.00mm_Vertical
- L1: footprint (none) -> Inductor_SMD:L_0402_1005Metric
- L2: footprint (none) -> Inductor_SMD:L_0805_2012Metric
- R1, R10, R5, R6, R7, R8, R9: footprint (none) -> Resistor_SMD:R_0402_1005Metric
- SW1: footprint (none) -> Button_Switch_SMD:SW_SPST_CK_RS282G05A3
- Y1: footprint (none) -> Crystal:Crystal_SMD_2012-2Pin_2.0x1.2mm
- Y2: footprint (none) -> Crystal:Crystal_SMD_2016-4Pin_2.0x1.6mm
Changed lines of the file:
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@@
 			)
 		)
-		(property "Footprint" ""
+		(property "Footprint" "Capacitor_SMD:C_0402_1005Metric"
 			(at 120.3452 31.75 0)
 			(effects
@@
 			)
 		)
-		(property "Footprint" ""
+		(property "Footprint" "LED_THT:LED_D3.0mm"
 			(at 180.34 144.78 0)
 			(effects
@@
 			)
 		)
-		(property "Footprint" ""
+		(property "Footprint" "Capacitor_SMD:C_0603_1608Metric"
 			(at 75.2348 63.5 0)
 			(effects
@@
 			)
 		)
-		(property "Footprint" ""
+		(property "Footprint" "Capacitor_SMD:C_0402_1005Metric"
 			(at 61.2648 60.96 0)
 			(effects
@@
 			)
 		)
-		(property "Footprint" ""
+		(property "Footprint" "Capacitor_SMD:C_0402_1005Metric"
 			(at 171.7548 30.48 0)
 			(effects
@@
 			)
 		)
-		(property "Footprint" ""
+		(property "Footprint" "Capacitor_SMD:C_0402_1005Metric"
 			(at 98.7552 52.07 0)
 			(effects
@@
 			)
 		)
-		(property "Footprint" ""
+		(property "Footprint" "Resistor_SMD:R_0402_1005Metric"
 			(at 46.482 157.48 90)
 			(effects
@@
 			)
 		)
-		(property "Footprint" ""
+		(property "Footprint" "Capacitor_SMD:C_0402_1005Metric"
 			(at 147.32 22.5552 0)
 			(effects
@@
 			)
 		)
-		(property "Footprint" ""
+		(property "Footprint" "Resistor_SMD:R_0402_1005Metric"
 			(at 151.892 153.67 90)
 			(effects
@@
 			)
 		)
-		(property "Footprint" ""
+		(property "Footprint" "Capacitor_SMD:C_0603_1608Metric"
 			(at 105.1052 91.44 0)
 			(effects
@@
 			)
 		)
-		(property "Footprint" ""
+		(property "Footprint" "Inductor_SMD:L_0805_2012Metric"
 			(at 104.14 77.47 0)
 			(effects
@@
 			)
 		)
-		(property "Footprint" ""
+		(property "Footprint" "Capacitor_SMD:C_0402_1005Metric"
 			(at 86.0552 142.24 0)
 			(effects
@@
 			)
 		)
-		(property "Footprint" ""
+		(property "Footprint" "Connector_PinHeader_1.00mm:PinHeader_1x04_P1.00mm_Vertical"
 			(at 184.15 87.63 0)
 			(effects
@@
 			)
 		)
-		(property "Footprint" ""
+		(property "Footprint" "Resistor_SMD:R_0402_1005Metric"
 			(at 195.072 138.43 90)
 			(effects
@@
 			)
 		)
-		(property "Footprint" ""
+		(property "Footprint" "Capacitor_SMD:C_0402_1005Metric"
 			(at 110.1852 31.75 0)
 			(effects
@@
 			)
 		)
-		(property "Footprint" ""
+		(property "Footprint" "LED_THT:LED_D3.0mm"
 			(at 168.91 144.78 0)
 			(effects
@@
 			)
 		)
-		(property "Footprint" ""
+		(property "Footprint" "Capacitor_SMD:C_0402_1005Metric"
 			(at 227.0252 123.19 0)
 			(effects
@@
 			)
 		)
-		(property "Footprint" ""
+		(property "Footprint" "Crystal:Crystal_SMD_2012-2Pin_2.0x1.2mm"
 			(at 97.79 132.08 0)
 			(effects
@@
 			)
 		)
-		(property "Footprint" ""
+		(property "Footprint" "Resistor_SMD:R_0402_1005Metric"
 			(at 167.132 153.67 90)
 			(effects
@@
 			)
 		)
-		(property "Footprint" ""
+		(property "Footprint" "Buzzer_Beeper:Buzzer_12x9.5RM7.6"
 			(at 240.665 20.32 90)
 			(effects
@@
 			)
 		)
-		(property "Footprint" ""
+		(property "Footprint" "Capacitor_SMD:C_0603_1608Metric"
 			(at 82.2452 31.75 0)
 			(effects
@@
 			)
 		)
-		(property "Footprint" ""
+		(property "Footprint" "Capacitor_SMD:C_0402_1005Metric"
 			(at 91.1352 31.75 0)
 			(effects
@@
 			)
 		)
-		(property "Footprint" ""
+		(property "Footprint" "LED_THT:LED_D3.0mm"
 			(at 153.67 144.78 0)
 			(effects
@@
 			)
 		)
-		(property "Footprint" ""
+		(property "Footprint" "Capacitor_SMD:C_0402_1005Metric"
 			(at 146.05 17.4752 0)
 			(effects
@@
 			)
 		)
-		(property "Footprint" ""
+		(property "Footprint" "Resistor_SMD:R_0402_1005Metric"
 			(at 206.502 138.43 90)
 			(effects
@@
 			)
 		)
-		(property "Footprint" ""
+		(property "Footprint" "Crystal:Crystal_SMD_2016-4Pin_2.0x1.6mm"
 			(at 85.09 82.55 0)
 			(effects
@@
 			)
 		)
-		(property "Footprint" ""
+		(property "Footprint" "Capacitor_SMD:C_0402_1005Metric"
 			(at 193.3448 26.67 0)
 			(effects
@@
 			)
 		)
-		(property "Footprint" ""
+		(property "Footprint" "Resistor_SMD:R_0402_1005Metric"
 			(at 215.9 29.972 90)
 			(effects
@@
 			)
 		)
-		(property "Footprint" ""
+		(property "Footprint" "Capacitor_SMD:C_0402_1005Metric"
 			(at 108.9152 143.51 0)
 			(effects
@@
 			)
 		)
-		(property "Footprint" ""
+		(property "Footprint" "Connector_PinHeader_1.00mm:PinHeader_1x04_P1.00mm_Vertical"
 			(at 187.96 45.72 0)
 			(effects
@@
 			)
 		)
-		(property "Footprint" ""
+		(property "Footprint" "Resistor_SMD:R_0402_1005Metric"
 			(at 178.562 153.67 90)
 			(effects
@@
 			)
 		)
-		(property "Footprint" ""
+		(property "Footprint" "Button_Switch_SMD:SW_SPST_CK_RS282G05A3"
 			(at 80.01 46.99 0)
 			(effects
@@
 			)
 		)
-		(property "Footprint" ""
+		(property "Footprint" "Capacitor_SMD:C_0402_1005Metric"
 			(at 100.0252 31.75 0)
 			(effects
@@
 			)
 		)
-		(property "Footprint" ""
+		(property "Footprint" "Inductor_SMD:L_0402_1005Metric"
 			(at 104.14 68.58 0)
 			(effects
@@
 			)
 		)
-		(property "Footprint" ""
+		(property "Footprint" "Capacitor_SMD:C_0603_1608Metric"
 			(at 202.2348 26.67 0)
 			(effects

Commit message: [FOOTPRINT ASSIGNMENT] : J'ai ajouté le +5V flag de l'USB, j'ai ajouté des labels pour avoir un netclass plus consistent
Connections:
- net RF SECTION/RF_IN renamed RF
- net USB SCHEME/USB_D+ renamed USB_D+
- net USB SCHEME/USB_D- renamed USB_D-
Changed lines of the file:
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@@
+		)
+	)
+	(label "USB_D-"
+		(at 177.8 55.88 0)
+		(effects
+			(font
+				(size 1.27 1.27)
+			)
+			(justify left bottom)
 		)
 	)
@@
 		)
 	)
+	(label "RF"
+		(at 76.2 109.22 0)
+		(effects
+			(font
+				(size 1.27 1.27)
+			)
+			(justify left bottom)
+		)
+	)
 	(label "SWDIO"
 		(at 172.72 78.74 0)
 		(effects
 			(font
+				(size 1.27 1.27)
+			)
+			(justify left bottom)
+		)
+	)
+	(label "USB_D+"
+		(at 179.07 60.96 0)
+		(effects
+			(font

Commit message: [VERIFICATION, CORRECTION DES FOOTPRINTS ET MODELES 3D, ET ETABLISSEMENT DES REGLES DE DESIGN DU PCB]
Le but de cette partie est de démarrer la phase du routage PCB.
Je concois un PCB 4 couches ici, et il y'a des montages hyperfrequences
donc il faut prendre en compte l'impédence de la ligne dans le design.
Il y'a également la ligne USB qui doit aussi etre une ligne 50 Ohm
adapté avec une impédance différentielle de 90 Ohm.
Une phase essentielle a été de calculer la largeur de la piste dans les
deux cas en utilisant les formules mathématique fournit par PCB Way
design. Le but ici est de trouver la largeur de la piste permettant
d'obtenir une impédance de ligne de 50 Ohm pour le montage RF, et une
impédance de ligne et une impédance différentielle de 90 Ohm pour le
montage USB.

Pendant la phase de vérification des modèles 3D de la carte, il y'a le
Microcontrolleur qui manquait, il y'avait également les deux crystals de
résonnance ainsi que le filter FLT1.
J'ai du utiliser snap magic et 3D Content Centrale pour avoir le modèle
3D nécessaire.

Enfin, j'ai fait 6 netclass :
1- PWR
2- GND
3- USB
4- RF
5- SWD
6- I2C

Les netclass permettent de faire le routage par montage et c'est plus
facile de se retrouver durant le routage.
Parts:
- U1: footprint Package_DFN_QFN:QFN-68-1EP_8x8mm_P0.4mm_EP6.4x6.4mm -> my_personnal_Library_footprint:QFN40P800X800X100-69N
Changed lines of the file:
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@@
 			)
 		)
-		(property "Footprint" "Package_DFN_QFN:QFN-68-1EP_8x8mm_P0.4mm_EP6.4x6.4mm"
+		(property "Footprint" "my_personnal_Library_footprint:QFN40P800X800X100-69N"
 			(at 121.92 132.08 0)
 			(effects

Commit message: [PLACEMENT DES COMPOSANT ET DIMENSIONNEMENT] : Avant de désigner le type de signal à chaque couche et commencer le routage, j'ai d'abord commencer par organiser les composants selon la schématique et comment j'aimerais avoir le produit finale
Connections:
- net RESET: now also C1.1
Changed lines of the file:
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@@
+	)
+	(junction
+		(at 97.79 41.91)
+		(diameter 0)
+		(color 0 0 0 0)
 	)
 	(junction
@@
 	(wire
 		(pts
+			(xy 107.95 41.91) (xy 107.95 45.72)
+		)
+		(stroke
+			(width 0)
+			(type default)
+		)
+	)
+	(wire
+		(pts
 			(xy 172.72 38.1) (xy 172.72 39.37)
 		)
@@
 	(wire
 		(pts
+			(xy 97.79 41.91) (xy 97.79 44.45)
+		)
+		(stroke
+			(width 0)
+			(type default)
+		)
+	)
+	(wire
+		(pts
 			(xy 100.33 82.55) (xy 100.33 60.96)
 		)
@@
 	(wire
 		(pts
-			(xy 97.79 45.72) (xy 119.38 45.72)
-		)
-		(stroke
-			(width 0)
-			(type default)
-		)
-	)
-	(wire
-		(pts
 			(xy 76.2 62.23) (xy 76.2 63.5)
 		)
@@
 	(wire
 		(pts
+			(xy 97.79 41.91) (xy 107.95 41.91)
+		)
+		(stroke
+			(width 0)
+			(type default)
+		)
+	)
+	(wire
+		(pts
 			(xy 62.23 62.23) (xy 62.23 60.96)
 		)
@@
 	(wire
 		(pts
-			(xy 97.79 41.91) (xy 97.79 45.72)
-		)
-		(stroke
+			(xy 107.95 45.72) (xy 119.38 45.72)
+		)
+		(stroke

Commit message: [Bill of Materials(BOM)]: Remplissage des informations tels que : manufacturer part number, manufacturer et la documentation du composant concerné. le BOM sera envoyé avec le fichier Geber au fabricant de PCB
Parts:
- BZ1: Manufacturer (none) -> Same Sky; Manufacturer Part Number (none) -> CMI-1295-85T
- C1, C12, C21, C3, C4, C5, C6, C7, C8, C9: Manufacturer (none) -> KYOCERA AVX; Manufacturer Part Number (none) -> 04023C104KAT2A
- C10: Manufacturer (none) -> KYOCERA AVX; Manufacturer Part Number (none) -> 04025A101JAT2A
- C11, C13, C2: Manufacturer (none) -> KYOCERA AVX; Manufacturer Part Number (none) -> 0603YD475MAT2A
- C14: Manufacturer (none) -> Murata Electronics; Manufacturer Part Number (none) -> GRM155R61E105KA12D
- C15, C16: Manufacturer (none) -> KYOCERA AVX; Manufacturer Part Number (none) -> 04025A100JAT4A
- D2: Manufacturer (none) -> Kingbright; Manufacturer Part Number (none) -> WP7113QBC/D
- D3: Manufacturer (none) -> Kingbright; Manufacturer Part Number (none) -> WP7113ND
- D4: Manufacturer (none) -> Kingbright; Manufacturer Part Number (none) -> WP7113SYD
- L1: Manufacturer (none) -> Murata Electronics; Manufacturer Part Number (none) -> LQG15WZ10NJ02D
- L2: Manufacturer (none) -> Murata Electronics; Manufacturer Part Number (none) -> LQM21FN100M70L
- Q1: Manufacturer (none) -> Diotec Semiconductor; Manufacturer Part Number (none) -> MMBT2222A
- R1: Manufacturer (none) -> YAGEO; Manufacturer Part Number (none) -> RC0402BR-0710KL
- R10, R8, R9: value 330 -> 220; Manufacturer (none) -> YAGEO; Manufacturer Part Number (none) -> RC0402FR-07221RL
- R5, R6: Manufacturer (none) -> YAGEO; Manufacturer Part Number (none) -> RC0402BR-074K7L
- R7: Manufacturer (none) -> YAGEO; Manufacturer Part Number (none) -> RC0402BR-071KL
- SW1: Manufacturer (none) -> C&K; Manufacturer Part Number (none) -> RS-282G05A3-SM RT
- U1: Manufacturer (none) -> STMicroelectronics; Manufacturer Part Number (none) -> STM32WB55RGV6
- U4: Manufacturer (none) -> Bosch Sensortec; Manufacturer Part Number (none) -> BME280
- Y1: Manufacturer (none) -> NDK; Manufacturer Part Number (none) -> NX2012SA-32.768K-STD-MUB-1
- Y2: Manufacturer (none) -> NDK; Manufacturer Part Number (none) -> NX2016SA-32M-EXS00A-CS06465

Commit message: [CORRECCTION DU PCB] : J'ai corrigé le PCB après avoir discuter avec le Fabricant PCB Way, j'ai corrigé le footprint de la capacité C14 avec ce qui correspond à ce qui est vendu par mouser electronics. Le bon footprint est 0402_1005. J'ai également corrigé le footprint des connecteurs 01x04 avec un footprint de 2.54mm. Avant c'était 1mm, du coup j'ai modifié le PCB. J'ai également modifier le placement des capacité et des inductances, plus proche du stm32.
Parts:
- C14: footprint Capacitor_SMD:C_0603_1608Metric -> Capacitor_SMD:C_0402_1005Metric
- J1, J4: footprint Connector_PinHeader_1.00mm:PinHeader_1x04_P1.00mm_Vertical -> Connector_PinHeader_2.54mm:PinHeader_1x04_P2.54mm_Vertical; Manufacturer (none) -> SAMTEC; Manufacturer Part Number (none) -> TSW-112-07-TM-S
Changed lines of the file:
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@@
 		(title "SAFE ROOM SCHEMATIC")
 		(date "2026-05-06")
-		(rev "0.1")
+		(rev "0.2")
 		(company "PAR KAMDA JONATAN")
 	)
@@
 			)
 		)
-		(property "Footprint" "Capacitor_SMD:C_0603_1608Metric"
+		(property "Footprint" "Capacitor_SMD:C_0402_1005Metric"
 			(at 75.2348 63.5 0)
 			(effects
@@
 			)
 		)
-		(property "Footprint" "Connector_PinHeader_1.00mm:PinHeader_1x04_P1.00mm_Vertical"
+		(property "Footprint" "Connector_PinHeader_2.54mm:PinHeader_1x04_P2.54mm_Vertical"
 			(at 184.15 87.63 0)
 			(effects
@@
 			)
 		)
-		(property "Datasheet" "~"
+		(property "Datasheet" "https://www.snapeda.com/parts/TSW-112-07-TM-S/Samtec/datasheet/"
 			(at 184.15 87.63 0)
 			(effects
@@
 			)
 		)
-		(property "Manufacturer" ""
+		(property "Manufacturer" "SAMTEC"
 			(at 184.15 87.63 90)
 			(effects
@@
 			)
 		)
-		(property "Manufacturer Part Number" ""
+		(property "Manufacturer Part Number" "TSW-112-07-TM-S "
 			(at 184.15 87.63 90)
 			(effects
@@
 			)
 		)
-		(property "Footprint" "Connector_PinHeader_1.00mm:PinHeader_1x04_P1.00mm_Vertical"
+		(property "Footprint" "Connector_PinHeader_2.54mm:PinHeader_1x04_P2.54mm_Vertical"
 			(at 187.96 45.72 0)
 			(effects
@@
 			)
 		)
-		(property "Datasheet" "~"
+		(property "Datasheet" "https://www.snapeda.com/parts/TSW-112-07-TM-S/Samtec/datasheet/"
 			(at 187.96 45.72 0)
 			(effects
@@
 			)
 		)
-		(property "Manufacturer" ""
+		(property "Manufacturer" "SAMTEC"
 			(at 187.96 45.72 0)
 			(effects
@@
 			)
 		)
-		(property "Manufacturer Part Number" ""
+		(property "Manufacturer Part Number" "TSW-112-07-TM-S "
 			(at 187.96 45.72 0)
 			(effects
